File: pcb/superlyra.kicad_pcb (KiCad board)
At the start: 2 copper layers, 391.1 x 134.8 mm, 199 parts, among them J1 USB_C_Receptacle_USB2.0, J2 AVR-ISP-6, SW1 SW_Push, SW10 SW_Push, SW11 SW_Push, SW12 SW_Push, SW13 SW_Push, SW14 SW_Push, SW15 SW_Push, SW16 SW_Push, SW17 SW_Push, SW18 SW_Push, SW19 SW_Push, SW2 SW_Push, SW20 SW_Push, SW21 SW_Push, SW22 SW_Push, SW23 SW_Push, SW24 SW_Push, SW25 SW_Push, SW26 SW_Push, SW27 SW_Push, SW28 SW_Push, SW29 SW_Push, SW3 SW_Push, SW30 SW_Push, SW31 SW_Push, SW32 SW_Push, SW33 SW_Push, SW34 SW_Push, SW35 SW_Push, SW36 SW_Push, SW37 SW_Push, SW38 SW_Push, SW39 SW_Push, SW4 SW_Push, SW40 SW_Push, SW41 SW_Push, SW42 SW_Push, SW43 SW_Push, SW44 SW_Push, SW45 SW_Push, SW46 SW_Push, SW47 SW_Push, SW48 SW_Push, SW49 SW_Push, SW5 SW_Push, SW50 SW_Push, SW51 SW_Push, SW52 SW_Push, SW53 SW_Push, SW54 SW_Push, SW55 SW_Push, SW56 SW_Push, SW57 SW_Push, SW58 SW_Push, SW59 SW_Push, SW6 SW_Push, SW60 SW_Push, SW61 SW_Push, SW62 SW_Push, SW63 SW_Push, SW64 SW_Push, SW65 SW_Push, SW66 SW_Push, SW67 SW_Push, SW68 SW_Push, SW69 SW_Push, SW7 SW_Push, SW70 SW_Push, SW71 SW_Push, SW72 SW_Push, SW73 SW_Push, SW74 SW_Push, SW75 SW_Push, SW76 SW_Push, SW77 SW_Push, SW78 SW_Push, SW79 SW_Push, SW8 SW_Push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

Commit message: update resonator
Parts:
- Y1: footprint Crystal:Crystal_SMD_3225-4Pin_3.2x2.5mm_HandSoldering -> Crystal:Resonator_SMD_muRata_CSTxExxV-3Pin_3.0x1.1mm_HandSoldering
- turned Y1 to 90 degrees
Routing:
- net GND: track 104.5 -> 113.4 mm

Commit message: Update superlyra.kicad_pcb
Parts:
- moved R3 4.06 mm to (227.3, 82.3), turned to 270 degrees
- moved C1 2.79 mm to (227.3, 80.3)
- moved C5 1.30 mm to (242.6, 80.0), turned to 0 degrees
Connections:
- J1 pad A1: GND1 -> GND
- J1 pad A12: GND1 -> GND
- J1 pad B1: GND1 -> GND
- J1 pad B12: GND1 -> GND
- J1 pad S1: GND1 -> GND
- U1 pad 5: GND1 -> GND
Routing:
- net GND1: track 54.1 -> 0.00 mm, vias 2 -> 0
- net Net-(C1-Pad1): track 11.2 -> 15.2 mm
- net RST: track 52.4 -> 56.4 mm
- net GND: track 113.4 -> 116.2 mm, vias 12 -> 8
- net COL16: track 185.1 -> 182.9 mm
- net COL17: track 203.7 -> 201.5 mm
- net COL15: track 167.6 -> 165.4 mm
- net COL14: track 145.3 -> 143.2 mm
- net COL13: track 122.7 -> 120.6 mm
- net VCC: track 129.7 -> 127.9 mm
- net COL12: track 105.3 -> 106.5 mm
- net Net-(U1-Pad17): track 13.5 -> 12.6 mm
- net Net-(U1-Pad16): track 10.8 -> 11.8 mm
- net ROW3: track 516.9 -> 517.8 mm
- net (no net): vias 1 -> 0
- added copper zone on B.Cu, net GND

Commit message: Update superlyra.kicad_pcb
Parts:
- moved C5 14.5 mm to (228.6, 83.8), turned to 270 degrees
- moved C2 13.6 mm to (243.3, 80.0), turned to 270 degrees
- moved C3 3.06 mm to (242.6, 90.2), turned to 270 degrees
- moved R4 2.34 mm to (241.3, 90.2), turned to 90 degrees
- moved Y1 2.05 mm to (226.1, 86.4)
Routing:
- net GND: track 116.2 -> 105.0 mm
- net MISO: track 449.3 -> 459.1 mm, vias 3 -> 6
- net MOSI: track 478.1 -> 486.0 mm, vias 5 -> 3
- net Net-(U1-Pad16): track 11.8 -> 7.27 mm
- net Net-(U1-Pad17): track 12.6 -> 8.77 mm
- net COL11: track 92.9 -> 95.0 mm
- net ROW4: track 517.9 -> 516.2 mm
- net RST: track 56.4 -> 55.3 mm
- net COL12: track 106.5 -> 107.6 mm
- net VCC: track 127.9 -> 126.9 mm, vias 8 -> 9
- net ROW0: track 404.5 -> 403.6 mm
- net ROW3: track 517.8 -> 518.2 mm, vias 3 -> 5

Commit message: Update superlyra.kicad_pcb
Routing:
- net MOSI: track 486.0 -> 511.3 mm
- net MISO: track 459.1 -> 482.3 mm
- net ROW3: track 518.2 -> 541.3 mm
- net VCC: track 126.9 -> 109.7 mm
- net GND: track 105.0 -> 88.7 mm, vias 8 -> 9
- net RST: track 55.3 -> 56.6 mm

Commit message: move diodes to front side
Parts:
- D1, D10, D11, D12, D13, D14, D15, D16, D17, D18, D19, D2, D20, D21, D22, D23, D24, D25, D26, D27, D28, D29, D3, D30, D31, D32, D33, D34, D35, D36, D37, D38, D39, D40, D41, D42, D43, D44, D45, D46, D47, D48, D49, D5, D50, D51, D52, D53, D54, D55, D56, D57, D58, D59, D6, D60, D61, D62, D63, D64, D65, D66, D67, D68, D69, D7, D70, D71, D72, D73, D74, D75, D76, D77, D78, D79, D8, D80, D81, D82, D83, D84, D85, D86, D87, D88, D89, D9, D90: moved to F.Cu
- Dr: renamed from D4; moved to F.Cu
- moved D79 17.1 mm to (171.2, 171.2), turned to 270 degrees
- moved D84 16.9 mm to (286.0, 166.1), turned to 270 degrees
- moved D21 12.1 mm to (90.9, 95.0), turned to 270 degrees
- moved D39 12.1 mm to (85.9, 113.5), turned to 270 degrees
- moved D74 12.1 mm to (57.1, 146.8), turned to 270 degrees
- moved D75 12.1 mm to (75.9, 150.4), turned to 270 degrees
- moved D37 11.8 mm to (49.0, 103.9), turned to 270 degrees
- moved D41 11.8 mm to (124.2, 117.6), turned to 270 degrees
- moved D43 11.8 mm to (160.0, 131.1), turned to 270 degrees
- moved D58 11.8 mm to (100.6, 132.3), turned to 270 degrees
- moved D59 11.8 mm to (119.4, 135.9), turned to 270 degrees
- moved D55 11.8 mm to (44.2, 122.2), turned to 270 degrees
- moved D56 11.8 mm to (62.2, 128.5), turned to 270 degrees
- moved D20 11.8 mm to (72.1, 91.7), turned to 270 degrees
- moved D22 11.8 mm to (110.5, 95.5), turned to 270 degrees
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Routing:
- net COL1: track 240.1 -> 207.4 mm
- net ROW4: track 516.2 -> 493.3 mm, vias 4 -> 2
- net MOSI: track 511.3 -> 489.6 mm, vias 3 -> 2
- net ROW3: track 541.3 -> 520.0 mm, vias 5 -> 4
- net MISO: track 482.3 -> 463.1 mm, vias 6 -> 5
- net ROW0: track 403.6 -> 389.3 mm, vias 1 -> 2
- net Net-(D90-Pad2): track 11.9 -> 3.46 mm
- net Net-(D19-Pad2): track 11.8 -> 4.17 mm
- net Net-(D80-Pad2): track 12.3 -> 4.95 mm
- net Net-(D82-Pad2): track 12.4 -> 5.04 mm
- net Net-(D81-Pad2): track 12.4 -> 5.00 mm
- net Net-(D49-Pad2): track 12.1 -> 4.71 mm
- net Net-(D48-Pad2): track 12.0 -> 4.63 mm
- net Net-(D26-Pad2): track 12.2 -> 4.91 mm
- net Net-(D62-Pad2): track 12.3 -> 4.98 mm
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
Commit message: front ground fill update
Routing:
- net GND: vias 9 -> 38
Changed lines of the file:
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@@
     (thickness 1.6)
     (drawings 18)
-    (tracks 1130)
+    (tracks 1159)
     (zones 0)
     (modules 199)
@@
   (segment (start 226.314 83.82) (end 226.314 83.82) (width 0.25) (layer F.Cu) (net 1))
   (via (at 226.314 83.82) (size 0.8) (drill 0.4) (layers F.Cu B.Cu) (net 1))
+  (via (at 59.436 72.644) (size 0.8) (drill 0.4) (layers F.Cu B.Cu) (net 1))
+  (via (at 78.232 76.2) (size 0.8) (drill 0.4) (layers F.Cu B.Cu) (net 1))
+  (via (at 97.536 77.978) (size 0.8) (drill 0.4) (layers F.Cu B.Cu) (net 1))
+  (via (at 116.84 79.756) (size 0.8) (drill 0.4) (layers F.Cu B.Cu) (net 1))
+  (via (at 135.382 83.312) (size 0.8) (drill 0.4) (layers F.Cu B.Cu) (net 1))
+  (via (at 153.162 89.916) (size 0.8) (drill 0.4) (layers F.Cu B.Cu) (net 1))
+  (via (at 173.228 94.996) (size 0.8) (drill 0.4) (layers F.Cu B.Cu) (net 1))
+  (via (at 192.532 96.266) (size 0.8) (drill 0.4) (layers F.Cu B.Cu) (net 1))
+  (via (at 210.566 96.012) (size 0.8) (drill 0.4) (layers F.Cu B.Cu) (net 1))
+  (via (at 230.124 96.266) (size 0.8) (drill 0.4) (layers F.Cu B.Cu) (net 1))
+  (via (at 250.952 96.012) (size 0.8) (drill 0.4) (layers F.Cu B.Cu) (net 1))
+  (via (at 270.002 95.758) (size 0.8) (drill 0.4) (layers F.Cu B.Cu) (net 1))
+  (via (at 282.448 93.472) (size 0.8) (drill 0.4) (layers F.Cu B.Cu) (net 1))
+  (via (at 288.798 90.17) (size 0.8) (drill 0.4) (layers F.Cu B.Cu) (net 1))
+  (via (at 297.942 89.662) (size 0.8) (drill 0.4) (layers F.Cu B.Cu) (net 1))
+  (via (at 307.086 81.788) (size 0.8) (drill 0.4) (layers F.Cu B.Cu) (net 1))
+  (via (at 326.39 81.28) (size 0.8) (drill 0.4) (layers F.Cu B.Cu) (net 1))
+  (via (at 339.598 83.566) (size 0.8) (drill 0.4) (layers F.Cu B.Cu) (net 1))
+  (via (at 344.17 77.47) (size 0.8) (drill 0.4) (layers F.Cu B.Cu) (net 1))
+  (via (at 358.648 79.756) (size 0.8) (drill 0.4) (layers F.Cu B.Cu) (net 1))
+  (via (at 362.204 73.66) (size 0.8) (drill 0.4) (layers F.Cu B.Cu) (net 1))
+  (via (at 375.92 73.406) (size 0.8) (drill 0.4) (layers F.Cu B.Cu) (net 1))
+  (via (at 302.514 95.504) (size 0.8) (drill 0.4) (layers F.Cu B.Cu) (net 1))
+  (via (at 286.766 98.298) (size 0.8) (drill 0.4) (layers F.Cu B.Cu) (net 1))
+  (via (at 273.304 102.87) (size 0.8) (drill 0.4) (layers F.Cu B.Cu) (net 1))
+  (via (at 211.074 110.49) (size 0.8) (drill 0.4) (layers F.Cu B.Cu) (net 1))
+  (via (at 106.934 93.726) (size 0.8) (drill 0.4) (layers F.Cu B.Cu) (net 1))
+  (via (at 230.886 91.186) (size 0.8) (drill 0.4) (layers F.Cu B.Cu) (net 1))
+  (via (at 218.186 83.312) (size 0.8) (drill 0.4) (layers F.Cu B.Cu) (net 1))
   (segment (start 237.744 78.428998) (end 237.744 79.067002) (width 0.25) (layer F.Cu) (net 2))
   (segment (start 237.293002 77.978) (end 237.744 78.428998) (width 0.25) (layer F.Cu) (net 2))

Commit message: Update superlyra.kicad_pcb
Parts:
- added G***: LOGO, gfx:SuperLyraLogo, F.Cu at (181.1, 84.3)
- added REF**: MountingHole_2.1mm, MountingHole:MountingHole_2.1mm, F.Cu at (142.2, 129.5)
- added REF**: MountingHole_2.1mm, MountingHole:MountingHole_2.1mm, F.Cu at (362.7, 78.7)
- added REF**: MountingHole_2.1mm, MountingHole:MountingHole_2.1mm, F.Cu at (303.8, 92.5)
- added REF**: MountingHole_2.1mm, MountingHole:MountingHole_2.1mm, F.Cu at (321.1, 145.0)
- added REF**: MountingHole_2.1mm, MountingHole:MountingHole_2.1mm, F.Cu at (378.7, 138.4)
- added REF**: MountingHole_2.1mm, MountingHole:MountingHole_2.1mm, F.Cu at (98.0, 147.3)
- added REF**: MountingHole_2.1mm, MountingHole:MountingHole_2.1mm, F.Cu at (114.3, 90.9)
- added REF**: MountingHole_2.1mm, MountingHole:MountingHole_2.1mm, F.Cu at (57.1, 78.7)
- added REF**: MountingHole_2.1mm, MountingHole:MountingHole_2.1mm, F.Cu at (41.7, 137.2)
- added REF**: MountingHole_2.1mm, MountingHole:MountingHole_2.1mm, F.Cu at (247.7, 78.7)
- added REF**: MountingHole_2.1mm, MountingHole:MountingHole_2.1mm, F.Cu at (172.7, 78.7)
- added REF**: MountingHole_2.1mm, MountingHole:MountingHole_2.1mm, F.Cu at (278.4, 132.1)
- added REF**: MountingHole_2.1mm, MountingHole:MountingHole_2.1mm, F.Cu at (229.1, 98.3)
- added REF**: MountingHole_2.1mm, MountingHole:MountingHole_2.1mm, F.Cu at (191.0, 98.3)
- added REF**: MountingHole_2.1mm, MountingHole:MountingHole_2.1mm, F.Cu at (229.1, 164.6)
- added REF**: MountingHole_2.1mm, MountingHole:MountingHole_2.1mm, F.Cu at (191.0, 164.6)
- added REF**: MountingHole_2.1mm, MountingHole:MountingHole_2.1mm, F.Cu at (210.1, 139.7)
- added REF**: MountingHole_2.1mm, MountingHole:MountingHole_2.1mm, F.Cu at (42.9, 61.2)
- added REF**: MountingHole_2.1mm, MountingHole:MountingHole_2.1mm, F.Cu at (376.9, 61.5)
- added REF**: MountingHole_2.1mm, MountingHole:MountingHole_2.1mm, F.Cu at (400.6, 149.1)
- added REF**: MountingHole_2.1mm, MountingHole:MountingHole_2.1mm, F.Cu at (19.3, 149.1)
- added REF**: MountingHole_2.1mm, MountingHole:MountingHole_2.1mm, F.Cu at (278.9, 188.0)
- added REF**: MountingHole_2.1mm, MountingHole:MountingHole_2.1mm, F.Cu at (141.0, 188.0)
- moved D79 21.5 mm to (152.4, 160.8)
- moved D84 17.8 mm to (268.2, 164.6)
- moved D13 3.31 mm to (288.8, 97.8)
- moved D14 3.31 mm to (306.8, 91.4)
- moved D17 3.31 mm to (364.0, 84.1)
- moved D18 3.31 mm to (382.0, 77.7)
- moved D12 3.31 mm to (271.0, 104.9)
- moved D15 3.31 mm to (325.6, 87.9)
- moved D16 2.96 mm to (345.2, 87.4)
- moved D3 2.70 mm to (90.7, 91.7)
- moved D1 2.70 mm to (53.8, 81.8)
- moved D6 2.70 mm to (147.1, 101.9)
- moved D7 2.70 mm to (164.8, 109.0)
- moved D2 2.54 mm to (72.1, 88.1)
- moved D4 2.54 mm to (110.5, 91.9)
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- renumbered Dr to D4
Routing:
- net COL1: track 207.4 -> 240.1 mm
- net ROW0: track 389.3 -> 402.5 mm
- net Net-(D12-Pad2): track 10.7 -> 20.2 mm
- net Net-(D84-Pad2): track 16.1 -> 7.14 mm
- net Net-(D14-Pad2): track 11.1 -> 19.9 mm
- net Net-(D17-Pad2): track 11.0 -> 18.7 mm
- net MISO: track 463.1 -> 469.7 mm, vias 5 -> 4
- net Net-(D13-Pad2): track 10.9 -> 16.5 mm
- net Net-(D7-Pad2): track 11.2 -> 15.8 mm
- net Net-(D6-Pad2): track 10.1 -> 14.6 mm
- net Net-(D2-Pad2): track 10.0 -> 14.4 mm
- net Net-(D3-Pad2): track 10.0 -> 14.3 mm
- net Net-(D4-Pad2): track 10.1 -> 14.4 mm
- net Net-(D15-Pad2): track 10.8 -> 15.1 mm
- net Net-(D5-Pad2): track 10.3 -> 14.4 mm
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Other:
- board text added: "by Domanic Calleja"
- board text added: "github.com/Malevolti/SuperLyra ver. 1.0 youtu.be/8CP6Chss0y0 Special thanks to Pat for know more about capacitors than me."
