File: pcb/superlyra.sch (KiCad schematic (older format))
At the start: 198 parts, among them J1 USB_C_Receptacle_USB2.0, J2 AVR-ISP-6, SW1 SW_Push, SW10 SW_Push, SW11 SW_Push, SW12 SW_Push, SW13 SW_Push, SW14 SW_Push, SW15 SW_Push, SW16 SW_Push, SW17 SW_Push, SW18 SW_Push, SW19 SW_Push, SW2 SW_Push, SW20 SW_Push, SW21 SW_Push, SW22 SW_Push, SW23 SW_Push, SW24 SW_Push, SW25 SW_Push, SW26 SW_Push, SW27 SW_Push, SW28 SW_Push, SW29 SW_Push, SW3 SW_Push, SW30 SW_Push, SW31 SW_Push, SW32 SW_Push, SW33 SW_Push, SW34 SW_Push, SW35 SW_Push, SW36 SW_Push, SW37 SW_Push, SW38 SW_Push, SW39 SW_Push, SW4 SW_Push, SW40 SW_Push, SW41 SW_Push, SW42 SW_Push, SW43 SW_Push, SW44 SW_Push, SW45 SW_Push, SW46 SW_Push, SW47 SW_Push, SW48 SW_Push, SW49 SW_Push, SW5 SW_Push, SW50 SW_Push, SW51 SW_Push, SW52 SW_Push, SW53 SW_Push, SW54 SW_Push, SW55 SW_Push, SW56 SW_Push, SW57 SW_Push, SW58 SW_Push, SW59 SW_Push, SW6 SW_Push, SW60 SW_Push, SW61 SW_Push, SW62 SW_Push, SW63 SW_Push, SW64 SW_Push, SW65 SW_Push, SW66 SW_Push, SW67 SW_Push, SW68 SW_Push, SW69 SW_Push, SW7 SW_Push, SW70 SW_Push, SW71 SW_Push, SW72 SW_Push, SW73 SW_Push, SW74 SW_Push, SW75 SW_Push, SW76 SW_Push, SW77 SW_Push, SW78 SW_Push, SW79 SW_Push, SW8 SW_Push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

Commit message: update resonator
Parts:
- Y1: footprint Crystal:Crystal_SMD_3225-4Pin_3.2x2.5mm_HandSoldering -> Crystal:Resonator_SMD_muRata_CSTxExxV-3Pin_3.0x1.1mm_HandSoldering
Changed lines of the file:
@@
 F 0 "Y1" V 4604 7160 50  0000 L CNN
 F 1 "16mhz" V 4695 7160 50  0000 L CNN
-F 2 "Crystal:Crystal_SMD_3225-4Pin_3.2x2.5mm_HandSoldering" H 4625 7050 50  0001 C CNN
+F 2 "Crystal:Resonator_SMD_muRata_CSTxExxV-3Pin_3.0x1.1mm_HandSoldering" H 4625 7050 50  0001 C CNN
 F 3 "~" H 4625 7050 50  0001 C CNN
 	1    4650 7050

Commit message: 0.5 (evaluation)
Parts:
- added C6: 0.1u, Keebio:C_0402, symbol Device:C_Small
- added H1, H10, H11, H12, H13, H14, H15, H16, H17, H18, H19, H2, H20, H21, H22, H23, H24, H3, H4, H5, H6, H7, H8, H9: MountingHole, MountingHole:MountingHole_2.2mm_M2_ISO7380_Pad, symbol Mechanical:MountingHole
- added H25: Logo, gfx:SuperLyraLogo, symbol Mechanical:MountingHole
- C1: LCSC (none) -> C106253
- C2, C3, C4: LCSC (none) -> C106204
- C5: LCSC (none) -> C237279
- D1, D10, D11, D12, D13, D14, D15, D16, D17, D18, D19, D2, D20, D21, D22, D23, D24, D25, D26, D27, D28, D29, D3, D30, D31, D32, D33, D34, D35, D36, D37, D38, D39, D4, D40, D41, D42, D43, D44, D45, D46, D47, D48, D49, D5, D50, D51, D52, D53, D54, D55, D56, D57, D58, D59, D6, D60, D61, D62, D63, D64, D65, D66, D67, D68, D69, D7, D70, D71, D72, D73, D74, D75, D76, D77, D78, D79, D8, D80, D81, D82, D83, D84, D85, D86, D87, D88, D89, D9, D90: footprint Keebio:D_0805 -> Diode_SMD:D_SOD-123F; LCSC (none) -> C2099
- F1: footprint Fuse:Fuse_1206_3216Metric -> Fuse:Fuse_0402_1005Metric; LCSC (none) -> C914085
- J1: LCSC (none) -> C165948
- R1, R2: LCSC (none) -> C93929
- R3, R4: LCSC (none) -> C60489
- R5, R6: LCSC (none) -> C25905
- SWRST1: LCSC (none) -> C318884
- U1: LCSC (none) -> C112161
- U2: LCSC (none) -> C558418
- Y1: LCSC (none) -> C341521
Connections:
- net GND1 is gone; now on net GND: J1.A1 (GND), J1.A12 (GND), J1.B1 (GND), J1.B12 (GND), J1.S1 (SHIELD), U1.5 (UGND)
- net GND: now also C6.2
- net VCC: now also C6.1
Other:
- moved on the sheet: C2, C3, C4
