File: pcb/hotswap/_autosave-superlyra-hs-plate.kicad_pcb (KiCad board)
At the start: 2 copper layers, 391.1 x 134.8 mm, 94 parts, among them J1 Conn_01x01_Female, SW1 SW_Push, SW12 SW_Push, SW13 SW_Push, SW14 SW_Push, SW15 SW_Push, SW16 SW_Push, SW17 SW_Push, SW18 SW_Push, SW19 SW_Push, SW2 SW_Push, SW20 SW_Push, SW21 SW_Push, SW22 SW_Push, SW23 SW_Push, SW24 SW_Push, SW25 SW_Push, SW3 SW_Push, SW30 SW_Push, SW31 SW_Push, SW32 SW_Push, SW33 SW_Push, SW34 SW_Push, SW35 SW_Push, SW36 SW_Push, SW37 SW_Push, SW38 SW_Push, SW39 SW_Push, SW4 SW_Push, SW40 SW_Push, SW41 SW_Push, SW42 SW_Push, SW43 SW_Push, SW44 SW_Push, SW45 SW_Push, SW46 SW_Push, SW47 SW_Push, SW48 SW_Push, SW49 SW_Push, SW5 SW_Push, SW50 SW_Push, SW51 SW_Push, SW52 SW_Push, SW53 SW_Push, SW54 SW_Push, SW55 SW_Push, SW56 SW_Push, SW57 SW_Push, SW58 SW_Push, SW59 SW_Push, SW6 SW_Push, SW60 SW_Push, SW61 SW_Push, SW62 SW_Push, SW65 SW_Push, SW66 SW_Push, SW67 SW_Push, SW68 SW_Push, SW69 SW_Push, SW7 SW_Push, SW70 SW_Push, SW71 SW_Push, SW72 SW_Push, SW73 SW_Push, SW74 SW_Push, SW75 SW_Push, SW76 SW_Push, SW77 SW_Push, SW78 SW_Push, SW79 SW_Push, SW80 SW_Push, SW81 SW_Push, SW82 SW_Push, SW83 SW_Push, SW84 SW_Push, SW85 SW_Push, SW86 SW_Push, SW87 SW_Push, SW88 SW_Push, SW89 SW_Push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

Commit message: Add Hotswap Ver
Parts:
- added G***: LOGO, gfx:bydomaniccallejasmallererpadver, F.Cu at (321.4, 173.4)
- added SW10: SW_Push, Keebio:MX_Switch_Cutout, F.Cu at (219.5, 101.7)
- added SW11: SW_Push, Keebio:MX_Switch_Cutout, F.Cu at (238.5, 101.7)
- added SW26: SW_Push, Keebio:MX_Switch_Cutout, F.Cu at (181.5, 120.7)
- added SW27: SW_Push, Keebio:MX_Switch_Cutout, F.Cu at (200.5, 120.7)
- added SW28: SW_Push, Keebio:MX_Switch_Cutout, F.Cu at (219.5, 120.7)
- added SW29: SW_Push, Keebio:MX_Switch_Cutout, F.Cu at (238.4, 120.7)
- added SW63: SW_Push, Keebio:MX_Switch_Cutout, F.Cu at (200.5, 158.7)
- added SW64: SW_Push, Keebio:MX_Switch_Cutout, F.Cu at (219.5, 158.7)
- added SW8: SW_Push, Keebio:MX_Switch_Cutout, F.Cu at (181.5, 101.7)
- added SW9: SW_Push, Keebio:MX_Switch_Cutout, F.Cu at (200.5, 101.7)
- H25: footprint gfx:SuperLyraLogo -> gfx:SuperLyraLogoblackmask-padver
- moved H25 0.74 mm to (209.7, 85.4)
- moved J1 0.40 mm to (209.8, 129.9)
