File: pcb/hotswap/superlyra-hs.kicad_pcb (KiCad board)
At the start: 2 copper layers, 391.1 x 134.8 mm, 212 parts, among them J1 USB_C_Receptacle_USB2.0, J2 AVR-ISP-6, SW1 SW_Push, SW10 SW_Push, SW11 SW_Push, SW12 SW_Push, SW13 SW_Push, SW14 SW_Push, SW15 SW_Push, SW16 SW_Push, SW17 SW_Push, SW18 SW_Push, SW19 SW_Push, SW2 SW_Push, SW20 SW_Push, SW21 SW_Push, SW22 SW_Push, SW23 SW_Push, SW24 SW_Push, SW25 SW_Push, SW26 SW_Push, SW27 SW_Push, SW28 SW_Push, SW29 SW_Push, SW3 SW_Push, SW30 SW_Push, SW31 SW_Push, SW32 SW_Push, SW33 SW_Push, SW34 SW_Push, SW35 SW_Push, SW36 SW_Push, SW37 SW_Push, SW38 SW_Push, SW39 SW_Push, SW4 SW_Push, SW40 SW_Push, SW41 SW_Push, SW42 SW_Push, SW43 SW_Push, SW44 SW_Push, SW45 SW_Push, SW46 SW_Push, SW47 SW_Push, SW48 SW_Push, SW49 SW_Push, SW5 SW_Push, SW50 SW_Push, SW51 SW_Push, SW52 SW_Push, SW53 SW_Push, SW54 SW_Push, SW55 SW_Push, SW56 SW_Push, SW57 SW_Push, SW58 SW_Push, SW59 SW_Push, SW6 SW_Push, SW60 SW_Push, SW61 SW_Push, SW62 SW_Push, SW63 SW_Push, SW64 SW_Push, SW65 SW_Push, SW66 SW_Push, SW67 SW_Push, SW68 SW_Push, SW69 SW_Push, SW7 SW_Push, SW70 SW_Push, SW71 SW_Push, SW72 SW_Push, SW73 SW_Push, SW74 SW_Push, SW75 SW_Push, SW76 SW_Push, SW77 SW_Push, SW78 SW_Push, SW79 SW_Push, SW8 SW_Push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

Commit message: Add Hotswap Ver
Parts:
- H25: footprint gfx:SuperLyraLogo -> gfx:SuperLyraLogoblackmask
- moved D84 17.8 mm to (285.8, 159.8)
Routing:
- net Net-(D84-Pad2): track 22.6 -> 44.8 mm
- net ROW0: track 370.5 -> 386.4 mm
- net MISO: track 429.8 -> 437.4 mm
- net ROW4: track 473.4 -> 479.1 mm
- net Net-(D86-Pad2): track 16.2 -> 21.6 mm
- net Net-(D71-Pad2): track 16.4 -> 21.2 mm
- net Net-(D31-Pad2): track 16.6 -> 21.2 mm
- net Net-(D69-Pad2): track 15.7 -> 20.2 mm
- net MOSI: track 455.6 -> 459.5 mm
- net Net-(D67-Pad2): track 16.6 -> 20.1 mm
- net Net-(D52-Pad2): track 16.1 -> 19.6 mm
- net Net-(D49-Pad2): track 16.6 -> 20.0 mm
- net ROW3: track 474.3 -> 477.6 mm
- net Net-(D48-Pad2): track 16.4 -> 19.8 mm
- net Net-(D85-Pad2): track 16.3 -> 19.6 mm
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- added copper zone on F.Cu, net (none)
